Commit message: Add placeholder inertia values to silence printing

File: src/pb_robot/models/franka_description/robots/panda_arm_hand.urdf (robot description, URDF)
Before this commit: robot panda, 13 links, 12 joints
Links:
- link panda_hand: mass None -> 0
- link panda_leftfinger: mass None -> 0
- link panda_link0: mass None -> 0
- link panda_link1: mass None -> 0
- link panda_link2: mass None -> 0
- link panda_link3: mass None -> 0
- link panda_link4: mass None -> 0
- link panda_link5: mass None -> 0
- link panda_link6: mass None -> 0
- link panda_link7: mass None -> 0
- link panda_link8: mass None -> 0
- link panda_rightfinger: mass None -> 0
- link tool_link: mass None -> 0

Commit message: Revert inertia entries, they mess up simulation

File: src/pb_robot/models/franka_description/robots/panda_arm_hand.urdf (robot description, URDF)
Before this commit: robot panda, 13 links, 12 joints
Links:
- link panda_hand: mass 0 -> None
- link panda_leftfinger: mass 0 -> None
- link panda_link0: mass 0 -> None
- link panda_link1: mass 0 -> None
- link panda_link2: mass 0 -> None
- link panda_link3: mass 0 -> None
- link panda_link4: mass 0 -> None
- link panda_link5: mass 0 -> None
- link panda_link6: mass 0 -> None
- link panda_link7: mass 0 -> None
- link panda_link8: mass 0 -> None
- link panda_rightfinger: mass 0 -> None
- link tool_link: mass 0 -> None
