Commit message: New Spot URDFS

File: src/pb_robot/models/spot_description/spot.urdf (robot description, URDF)
Before this commit: robot spot, 21 links, 20 joints
Links:
- removed link arm0.link_el0
- removed link arm0.link_el1
- removed link arm0.link_fngr
- removed link arm0.link_hr0
- removed link arm0.link_sh0
- removed link arm0.link_sh1
- removed link arm0.link_wr0
- removed link arm0.link_wr1
- removed link base
- removed link fl.hip
- removed link fl.lleg
- removed link fl.uleg
- removed link fr.hip
- removed link fr.lleg
- removed link fr.uleg
- removed link hl.hip
- removed link hl.lleg
- removed link hl.uleg
- removed link hr.hip
- removed link hr.lleg
- removed link hr.uleg
- added link arm_link_el0, mass 0.725; collision mesh filename=meshes/arm/collision/arm_link_el0.stl; visual mesh filename=meshes/arm/visual/arm_link_el0.obj
- added link arm_link_el1, mass 0.725; collision mesh filename=meshes/arm/collision/arm_link_el1.stl; visual mesh filename=meshes/arm/visual/arm_link_el1.obj
- added link arm_link_fngr, mass 0.2; collision mesh filename=meshes/arm/collision/arm_link_fngr.stl; visual mesh filename=meshes/arm/visual/arm_link_fngr.obj
- added link arm_link_hr0, mass 1e-06; collision mesh filename=meshes/arm/collision/arm_link_hr0.stl; visual mesh filename=meshes/arm/visual/arm_link_hr0.obj
- added link arm_link_sh0, mass 2.3364000000000003; collision mesh filename=meshes/arm/collision/arm_link_sh0.stl; visual mesh filename=meshes/arm/visual/arm_link_sh0.obj
- added link arm_link_sh1, mass 0.2596; collision mesh filename=meshes/arm/collision/arm_link_sh1.stl; visual mesh filename=meshes/arm/visual/arm_link_sh1.obj
- added link arm_link_wr0, mass 0.98; collision mesh filename=meshes/arm/collision/arm_link_wr0.stl; visual mesh filename=meshes/arm/visual/arm_link_wr0.obj
- added link arm_link_wr1, mass 0.785; collision mesh filename=meshes/arm/collision/arm_link_wr1.stl; visual mesh filename=meshes/arm/visual/arm_link_wr1.obj
- added link body; collision mesh filename=meshes/base_simple/collision/body.stl; visual mesh filename=meshes/base_simple/visual/body.obj
- added link body_inertia, mass 32.86
- added link fl_hip, mass 1.68; collision mesh filename=meshes/base_simple/collision/fl_hip.stl; visual mesh filename=meshes/base_simple/visual/fl_hip.obj
- added link fl_lleg, mass 0.35; collision mesh filename=meshes/base_simple/collision/fl_lleg.stl; visual mesh filename=meshes/base_simple/visual/fl_lleg.obj
- added link fl_uleg, mass 2.34; collision mesh filename=meshes/base_simple/collision/fl_uleg.stl; visual mesh filename=meshes/base_simple/visual/fl_uleg.obj
- added link fr_hip, mass 1.68; collision mesh filename=meshes/base_simple/collision/fr_hip.stl; visual mesh filename=meshes/base_simple/visual/fr_hip.obj
- added link fr_lleg, mass 0.35; collision mesh filename=meshes/base_simple/collision/fr_lleg.stl; visual mesh filename=meshes/base_simple/visual/fr_lleg.obj
- added link fr_uleg, mass 2.34; collision mesh filename=meshes/base_simple/collision/fr_uleg.stl; visual mesh filename=meshes/base_simple/visual/fr_uleg.obj
- added link hl_hip, mass 1.68; collision mesh filename=meshes/base_simple/collision/hl_hip.stl; visual mesh filename=meshes/base_simple/visual/hl_hip.obj
- added link hl_lleg, mass 0.35; collision mesh filename=meshes/base_simple/collision/hl_lleg.stl; visual mesh filename=meshes/base_simple/visual/hl_lleg.obj
- added link hl_uleg, mass 2.34; collision mesh filename=meshes/base_simple/collision/hl_uleg.stl; visual mesh filename=meshes/base_simple/visual/hl_uleg.obj
- added link hr_hip, mass 1.68; collision mesh filename=meshes/base_simple/collision/hr_hip.stl; visual mesh filename=meshes/base_simple/visual/hr_hip.obj
- added link hr_lleg, mass 0.35; collision mesh filename=meshes/base_simple/collision/hr_lleg.stl; visual mesh filename=meshes/base_simple/visual/hr_lleg.obj
- added link hr_uleg, mass 2.34; collision mesh filename=meshes/base_simple/collision/hr_uleg.stl; visual mesh filename=meshes/base_simple/visual/hr_uleg.obj
Joints:
- removed joint arm0.el0
- removed joint arm0.el1
- removed joint arm0.f1x
- removed joint arm0.hr0
- removed joint arm0.sh0
- removed joint arm0.sh1
- removed joint arm0.wr0
- removed joint arm0.wr1
- removed joint fl.hx
- removed joint fl.hy
- removed joint fl.kn
- removed joint fr.hx
- removed joint fr.hy
- removed joint fr.kn
- removed joint hl.hx
- removed joint hl.hy
- removed joint hl.kn
- removed joint hr.hx
- removed joint hr.hy
- removed joint hr.kn
- added joint arm_el0: type revolute, parent arm_link_hr0, child arm_link_el0, origin xyz=0.3385 0 0 rpy=0 0 0, axis 0 1 0, limit lower=0 upper=3.14159265358979311599 effort=1000 velocity=1000.00
- added joint arm_el1: type revolute, parent arm_link_el0, child arm_link_el1, origin xyz=0.40330 0.0 0.0750 rpy=0 0 0, axis 1 0 0, limit lower=-2.79252680319092716487 upper=2.79252680319092716487 effort=1000 velocity=1000.00
- added joint arm_f1x: type revolute, parent arm_link_wr1, child arm_link_fngr, origin xyz=0.11745 0 0.014820 rpy=0 0 0, axis 0.0 1.0 0.0, limit lower=-1.57 upper=0.0 effort=1000 velocity=1000.00
- added joint arm_hr0: type fixed, parent arm_link_sh1, child arm_link_hr0, origin xyz=0.0 0.0 0.0 rpy=0 0 0, axis 1 0 0, limit lower=-1e6 upper=1e6 effort=1000 velocity=1000.00
- added joint arm_sh0: type revolute, parent body, child arm_link_sh0, origin xyz=0.292 0.0 0.188 rpy=0 0 0, axis 0 0 1, limit lower=-2.61799387799149441136 upper=3.14159265358979311599 effort=1000 velocity=1000.00
- added joint arm_sh1: type revolute, parent arm_link_sh0, child arm_link_sh1, origin xyz=0.0 0.0 0.0 rpy=0 0 0, axis 0 1 0, limit lower=-3.14159265358979311599 upper=0.52359877559829881565 effort=1000 velocity=1000.00
- added joint arm_wr0: type revolute, parent arm_link_el1, child arm_link_wr0, origin xyz=0.0 0.0 0.0 rpy=0 0 0, axis 0 1 0, limit lower=-1.83259571459404613236 upper=1.83259571459404613236 effort=1000 velocity=1000.00
- added joint arm_wr1: type revolute, parent arm_link_wr0, child arm_link_wr1, origin xyz=0.0 0.0 0.0 rpy=0 0 0, axis 1 0 0, limit lower=-2.87979326579064354163 upper=2.87979326579064354163 effort=1000 velocity=1000.00
- added joint body_inertia_joint: type fixed, parent body, child body_inertia, origin xyz=0 0 0 rpy=0 0 0
- added joint fl_hx: type revolute, parent body, child fl_hip, origin xyz=0.29785 0.05500 0.00000 rpy=0 0 0, axis 1 0 0, limit lower=-0.78539816339744827899 upper=0.78539816339744827899 effort=1000 velocity=1000.00
- added joint fl_hy: type revolute, parent fl_hip, child fl_uleg, origin xyz=0.0 0.11080 0.0 rpy=0 0 0, axis 0 1      0, limit lower=-0.89884456477707963539 upper=2.2951079663725435509 effort=1000 velocity=1000.00
- added joint fl_kn: type revolute, parent fl_uleg, child fl_lleg, origin xyz=0.025 0.000 -0.3200 rpy=0 0 0, axis 0 1 0, limit lower=-2.7929 upper=-0.254402 effort=1000 velocity=1000.00
- added joint fr_hx: type revolute, parent body, child fr_hip, origin xyz=0.29785 -0.05500 0.00000 rpy=0 0 0, axis 1 0 0, limit lower=-0.78539816339744827899 upper=0.78539816339744827899 effort=1000 velocity=1000.00
- added joint fr_hy: type revolute, parent fr_hip, child fr_uleg, origin xyz=0.0 -0.11080 0.0 rpy=0 0 0, axis 0  1      0, limit lower=-0.898845 upper=2.24363 effort=1000 velocity=1000.00
- added joint fr_kn: type revolute, parent fr_uleg, child fr_lleg, origin xyz=0.025 0.000 -0.3200 rpy=0 0 0, axis 0 1 0, limit lower=-2.7929 upper=-0.255648 effort=1000 velocity=1000.00
- added joint hl_hx: type revolute, parent body, child hl_hip, origin xyz=-0.29785 0.05500 0.00000 rpy=0 0 0, axis 1 0 0, limit lower=-0.78539816339744827899 upper=0.78539816339744827899 effort=1000 velocity=1000.00
- added joint hl_hy: type revolute, parent hl_hip, child hl_uleg, origin xyz=0.0 0.11080 0.0 rpy=0 0 0, axis 0 1      0, limit lower=-0.89884456477707963539 upper=2.2951079663725435509 effort=1000 velocity=1000.00
- added joint hl_kn: type revolute, parent hl_uleg, child hl_lleg, origin xyz=0.025 0.000 -0.3200 rpy=0 0 0, axis 0 1 0, limit lower=-2.7929 upper=-0.247067 effort=1000 velocity=1000.00
- added joint hr_hx: type revolute, parent body, child hr_hip, origin xyz=-0.29785 -0.05500 0.00000 rpy=0 0 0, axis 1 0 0, limit lower=-0.78539816339744827899 upper=0.78539816339744827899 effort=1000 velocity=1000.00
- added joint hr_hy: type revolute, parent hr_hip, child hr_uleg, origin xyz=0.0 -0.11080 0.0 rpy=0 0 0, axis 0  1      0, limit lower=-0.89884456477707963539 upper=2.2951079663725435509 effort=1000 velocity=1000.00
- added joint hr_kn: type revolute, parent hr_uleg, child hr_lleg, origin xyz=0.025 0.000 -0.3200 rpy=0 0 0, axis 0 1 0, limit lower=-2.7929 upper=-0.248282 effort=1000 velocity=1000.00

File: src/pb_robot/models/spot_description/spot_arm.urdf (robot description, URDF)
Before this commit: robot spot, 9 links, 8 joints
Links:
- removed link arm0.link_el0
- removed link arm0.link_el1
- removed link arm0.link_fngr
- removed link arm0.link_hr0
- removed link arm0.link_sh0
- removed link arm0.link_sh1
- removed link arm0.link_wr0
- removed link arm0.link_wr1
- removed link base
- added link arm_link_el0, mass 0.725; collision mesh filename=meshes/arm/collision/arm_link_el0.stl; visual mesh filename=meshes/arm/visual/arm_link_el0.obj
- added link arm_link_el1, mass 0.725; collision mesh filename=meshes/arm/collision/arm_link_el1.stl; visual mesh filename=meshes/arm/visual/arm_link_el1.obj
- added link arm_link_fngr, mass 0.2; collision mesh filename=meshes/arm/collision/arm_link_fngr.stl; visual mesh filename=meshes/arm/visual/arm_link_fngr.obj
- added link arm_link_hr0, mass 1e-06; collision mesh filename=meshes/arm/collision/arm_link_hr0.stl; visual mesh filename=meshes/arm/visual/arm_link_hr0.obj
- added link arm_link_sh0, mass 2.3364000000000003; collision mesh filename=meshes/arm/collision/arm_link_sh0.stl; visual mesh filename=meshes/arm/visual/arm_link_sh0.obj
- added link arm_link_sh1, mass 0.2596; collision mesh filename=meshes/arm/collision/arm_link_sh1.stl; visual mesh filename=meshes/arm/visual/arm_link_sh1.obj
- added link arm_link_wr0, mass 0.98; collision mesh filename=meshes/arm/collision/arm_link_wr0.stl; visual mesh filename=meshes/arm/visual/arm_link_wr0.obj
- added link arm_link_wr1, mass 0.785; collision mesh filename=meshes/arm/collision/arm_link_wr1.stl; visual mesh filename=meshes/arm/visual/arm_link_wr1.obj
- added link body; collision mesh filename=meshes/base_simple/collision/body.stl; visual mesh filename=meshes/base_simple/visual/body.obj
- added link body_inertia, mass 32.86
Joints:
- removed joint arm0.el0
- removed joint arm0.el1
- removed joint arm0.f1x
- removed joint arm0.hr0
- removed joint arm0.sh0
- removed joint arm0.sh1
- removed joint arm0.wr0
- removed joint arm0.wr1
- added joint arm_el0: type revolute, parent arm_link_hr0, child arm_link_el0, origin xyz=0.3385 0 0 rpy=0 0 0, axis 0 1 0, limit lower=0 upper=3.14159265358979311599 effort=1000 velocity=1000.00
- added joint arm_el1: type revolute, parent arm_link_el0, child arm_link_el1, origin xyz=0.40330 0.0 0.0750 rpy=0 0 0, axis 1 0 0, limit lower=-2.79252680319092716487 upper=2.79252680319092716487 effort=1000 velocity=1000.00
- added joint arm_f1x: type revolute, parent arm_link_wr1, child arm_link_fngr, origin xyz=0.11745 0 0.014820 rpy=0 0 0, axis 0.0 1.0 0.0, limit lower=-1.57 upper=0.0 effort=1000 velocity=1000.00
- added joint arm_hr0: type fixed, parent arm_link_sh1, child arm_link_hr0, origin xyz=0.0 0.0 0.0 rpy=0 0 0, axis 1 0 0, limit lower=-1e6 upper=1e6 effort=1000 velocity=1000.00
- added joint arm_sh0: type revolute, parent body, child arm_link_sh0, origin xyz=0.292 0.0 0.188 rpy=0 0 0, axis 0 0 1, limit lower=-2.61799387799149441136 upper=3.14159265358979311599 effort=1000 velocity=1000.00
- added joint arm_sh1: type revolute, parent arm_link_sh0, child arm_link_sh1, origin xyz=0.0 0.0 0.0 rpy=0 0 0, axis 0 1 0, limit lower=-3.14159265358979311599 upper=0.52359877559829881565 effort=1000 velocity=1000.00
- added joint arm_wr0: type revolute, parent arm_link_el1, child arm_link_wr0, origin xyz=0.0 0.0 0.0 rpy=0 0 0, axis 0 1 0, limit lower=-1.83259571459404613236 upper=1.83259571459404613236 effort=1000 velocity=1000.00
- added joint arm_wr1: type revolute, parent arm_link_wr0, child arm_link_wr1, origin xyz=0.0 0.0 0.0 rpy=0 0 0, axis 1 0 0, limit lower=-2.87979326579064354163 upper=2.87979326579064354163 effort=1000 velocity=1000.00
- added joint body_inertia_joint: type fixed, parent body, child body_inertia, origin xyz=0 0 0 rpy=0 0 0

Commit message: New Spot URDFS

File: src/pb_robot/models/spot_description/spot.urdf (robot description, URDF)
Before this commit: robot spot, 22 links, 21 joints
Links:
- added link arm_end_effector_link
- added link world_link; visual box size=0.001 0.001 0.001
Joints:
- added joint base_joint: type fixed, parent world_link, child body, origin xyz=0 0 0.685 rpy=0 0 0
- added joint end_effector_joint: type fixed, parent arm_link_wr1, child arm_end_effector_link, origin xyz=0.25 0.0 0.0 rpy=-1.5707963267948966 0. 1.5707963267948966

File: src/pb_robot/models/spot_description/spot_arm.urdf (robot description, URDF)
Before this commit: robot spot, 10 links, 9 joints
Links:
- added link arm_end_effector_link
- added link world_link; visual box size=0.001 0.001 0.001
Joints:
- added joint base_joint: type fixed, parent world_link, child body, origin xyz=0 0 0.685 rpy=0 0 0
- added joint end_effector_joint: type fixed, parent arm_link_wr1, child arm_end_effector_link, origin xyz=0.25 0.0 0.0 rpy=-1.5707963267948966 0. 1.5707963267948966
